Commit message: Simulation of holding a tray working.

File: assets/fetch/fetch.urdf (robot description, URDF)
Before this commit: robot fetch, 20 links, 19 joints
Joints:
- joint head_pan_joint: type revolute -> fixed
- joint head_tilt_joint: type revolute -> fixed
- joint l_wheel_joint: type continuous -> fixed
- joint r_wheel_joint: type continuous -> fixed

File: assets/objects/cube_small.urdf (robot description, URDF)
Before this commit: robot cube.urdf, 1 links, 0 joints
Links:
- link baseLink: mass .1 -> .25
