Commit message: Rendering for matlab simulation working.

File: assets/fetch/fetch_arm_new_dumbbell.urdf (robot description, URDF)
Before this commit: robot fetch_arm, 13 links, 12 joints
Links:
- added link base
Joints:
- added joint translation: type fixed, parent base, child base_link, origin xyz=-0.06525 0 0
- joint shoulder_pan_joint: origin xyz=0.119525 0 0.34858 rpy=0 0 0 -> xyz=-0.0326 0 0.726 rpy=0 0 0; parent torso_lift_link -> base
