Commit message: update new demo for Amazon robotics

File: assets/fetch/fetch_waiter.urdf (robot description, URDF)
Before this commit: robot fetch_waiter_Zac, 10 links, 9 joints
Links:
- removed link base
- added link base_link, mass 70.1294; collision mesh filename=./meshes/base_link_collision.STL; visual mesh filename=./meshes/base_link.obj
- added link head_pan_link, mass 2.2556; collision mesh filename=./meshes/head_pan_link_collision.STL; visual mesh filename=./meshes/head_pan_link.obj
- added link head_tilt_link, mass 0.9087; collision mesh filename=./meshes/head_tilt_link_collision.STL; visual mesh filename=./meshes/head_tilt_link.obj
- added link l_wheel_link, mass 4.3542; collision mesh filename=./meshes/l_wheel_link_collision.STL; visual mesh filename=./meshes/l_wheel_link.STL
- added link r_wheel_link, mass 4.3542; collision mesh filename=./meshes/r_wheel_link_collision.STL; visual mesh filename=./meshes/r_wheel_link.STL
- added link torso_lift_link, mass 0; collision mesh filename=meshes/torso_lift_link_collision.STL; visual mesh filename=meshes/torso_lift_link.obj
Joints:
- added joint head_pan_joint: type fixed, parent torso_lift_link, child head_pan_link, origin xyz=0.053125 0 0.603001417713939 rpy=0 0 0, axis 0 0 1, limit lower=-1.57 upper=1.57 effort=0.32 velocity=1.57
- added joint head_tilt_joint: type fixed, parent head_pan_link, child head_tilt_link, origin xyz=0.14253 0 0.057999 rpy=0 0 0, axis 0 1 0, limit lower=-0.76 upper=1.45 effort=0.68 velocity=1.57
- added joint l_wheel_joint: type fixed, parent base_link, child l_wheel_link, origin xyz=0.0012914 0.18738 0.055325 rpy=-6.123E-17 0 0, axis 0 1 0, limit effort=8.85 velocity=17.4
- added joint r_wheel_joint: type fixed, parent base_link, child r_wheel_link, origin xyz=0.0012914 -0.18738 0.055325 rpy=-6.123E-17 0 0, axis 0 1 0, limit effort=8.85 velocity=17.4
- added joint torso_lift_joint: type fixed, parent base_link, child torso_lift_link, origin xyz=-0.086875 0 0.37743 rpy=-6.123E-17 0 0, axis 0 0 1, limit lower=0 upper=0.38615 effort=450.0 velocity=0.1
- joint shoulder_pan_joint: origin xyz=0 0 0 rpy=0 0 0 -> xyz=0.119525 0 0.34858 rpy=0 0 0; parent base -> torso_lift_link
