Commit message: Saving seperate .pkl file for Blender. Transform obj to urdf.

File: zonotope/_prototype.urdf (robot description, URDF)
Before this commit: robot _name, 1 links, 0 joints
Links:
- removed link 
- added link link0, mass 0; visual mesh filename=_prototype.obj scale=1.0 1.0 1.0

File: zonotope/meshes/zonopy_mesh_step10_link1_num1.obj.urdf (robot description, URDF)
Before this commit: robot zonopy_mesh_step10_link1_num1.obj, 1 links, 0 joints
Links:
- removed link 
- added link link0, mass 0; collision mesh filename=zonopy_mesh_step10_link1_num1.obj; visual mesh filename=zonopy_mesh_step10_link1_num1.obj scale=1.0 1.0 1.0

File: zonotope/meshes/zonopy_mesh_step10_link1_num2.obj.urdf (robot description, URDF)
Before this commit: robot zonopy_mesh_step10_link1_num2.obj, 1 links, 0 joints
Links:
- removed link 
- added link link0, mass 0; collision mesh filename=zonopy_mesh_step10_link1_num2.obj; visual mesh filename=zonopy_mesh_step10_link1_num2.obj scale=1.0 1.0 1.0

File: zonotope/meshes/zonopy_mesh_step10_link1_num3.obj.urdf (robot description, URDF)
Before this commit: robot zonopy_mesh_step10_link1_num3.obj, 1 links, 0 joints
Links:
- removed link 
- added link link0, mass 0; collision mesh filename=zonopy_mesh_step10_link1_num3.obj; visual mesh filename=zonopy_mesh_step10_link1_num3.obj scale=1.0 1.0 1.0

File: zonotope/meshes/zonopy_mesh_step10_link1_num4.obj.urdf (robot description, URDF)
Before this commit: robot zonopy_mesh_step10_link1_num4.obj, 1 links, 0 joints
Links:
- removed link 
- added link link0, mass 0; collision mesh filename=zonopy_mesh_step10_link1_num4.obj; visual mesh filename=zonopy_mesh_step10_link1_num4.obj scale=1.0 1.0 1.0

File: zonotope/meshes/zonopy_mesh_step10_link2_num1.obj.urdf (robot description, URDF)
Before this commit: robot zonopy_mesh_step10_link2_num1.obj, 1 links, 0 joints
Links:
- removed link 
- added link link0, mass 0; collision mesh filename=zonopy_mesh_step10_link2_num1.obj; visual mesh filename=zonopy_mesh_step10_link2_num1.obj scale=1.0 1.0 1.0

File: zonotope/meshes/zonopy_mesh_step10_link2_num2.obj.urdf (robot description, URDF)
Before this commit: robot zonopy_mesh_step10_link2_num2.obj, 1 links, 0 joints
Links:
- removed link 
- added link link0, mass 0; collision mesh filename=zonopy_mesh_step10_link2_num2.obj; visual mesh filename=zonopy_mesh_step10_link2_num2.obj scale=1.0 1.0 1.0

File: zonotope/meshes/zonopy_mesh_step10_link2_num3.obj.urdf (robot description, URDF)
Before this commit: robot zonopy_mesh_step10_link2_num3.obj, 1 links, 0 joints
Links:
- removed link 
- added link link0, mass 0; collision mesh filename=zonopy_mesh_step10_link2_num3.obj; visual mesh filename=zonopy_mesh_step10_link2_num3.obj scale=1.0 1.0 1.0

File: zonotope/meshes/zonopy_mesh_step10_link2_num4.obj.urdf (robot description, URDF)
Before this commit: robot zonopy_mesh_step10_link2_num4.obj, 1 links, 0 joints
Links:
- removed link 
- added link link0, mass 0; collision mesh filename=zonopy_mesh_step10_link2_num4.obj; visual mesh filename=zonopy_mesh_step10_link2_num4.obj scale=1.0 1.0 1.0

File: zonotope/meshes/zonopy_mesh_step10_link3_num1.obj.urdf (robot description, URDF)
Before this commit: robot zonopy_mesh_step10_link3_num1.obj, 1 links, 0 joints
Links:
- removed link 
- added link link0, mass 0; collision mesh filename=zonopy_mesh_step10_link3_num1.obj; visual mesh filename=zonopy_mesh_step10_link3_num1.obj scale=1.0 1.0 1.0

File: zonotope/meshes/zonopy_mesh_step10_link3_num2.obj.urdf (robot description, URDF)
Before this commit: robot zonopy_mesh_step10_link3_num2.obj, 1 links, 0 joints
Links:
- removed link 
- added link link0, mass 0; collision mesh filename=zonopy_mesh_step10_link3_num2.obj; visual mesh filename=zonopy_mesh_step10_link3_num2.obj scale=1.0 1.0 1.0

File: zonotope/meshes/zonopy_mesh_step10_link3_num3.obj.urdf (robot description, URDF)
Before this commit: robot zonopy_mesh_step10_link3_num3.obj, 1 links, 0 joints
Links:
- removed link 
- added link link0, mass 0; collision mesh filename=zonopy_mesh_step10_link3_num3.obj; visual mesh filename=zonopy_mesh_step10_link3_num3.obj scale=1.0 1.0 1.0

File: zonotope/meshes/zonopy_mesh_step10_link3_num4.obj.urdf (robot description, URDF)
Before this commit: robot zonopy_mesh_step10_link3_num4.obj, 1 links, 0 joints
Links:
- removed link 
- added link link0, mass 0; collision mesh filename=zonopy_mesh_step10_link3_num4.obj; visual mesh filename=zonopy_mesh_step10_link3_num4.obj scale=1.0 1.0 1.0

File: zonotope/meshes/zonopy_mesh_step10_link4_num1.obj.urdf (robot description, URDF)
Before this commit: robot zonopy_mesh_step10_link4_num1.obj, 1 links, 0 joints
Links:
- removed link 
- added link link0, mass 0; collision mesh filename=zonopy_mesh_step10_link4_num1.obj; visual mesh filename=zonopy_mesh_step10_link4_num1.obj scale=1.0 1.0 1.0

File: zonotope/meshes/zonopy_mesh_step10_link4_num2.obj.urdf (robot description, URDF)
Before this commit: robot zonopy_mesh_step10_link4_num2.obj, 1 links, 0 joints
Links:
- removed link 
- added link link0, mass 0; collision mesh filename=zonopy_mesh_step10_link4_num2.obj; visual mesh filename=zonopy_mesh_step10_link4_num2.obj scale=1.0 1.0 1.0

File: zonotope/meshes/zonopy_mesh_step10_link4_num3.obj.urdf (robot description, URDF)
Before this commit: robot zonopy_mesh_step10_link4_num3.obj, 1 links, 0 joints
Links:
- removed link 
- added link link0, mass 0; collision mesh filename=zonopy_mesh_step10_link4_num3.obj; visual mesh filename=zonopy_mesh_step10_link4_num3.obj scale=1.0 1.0 1.0

File: zonotope/meshes/zonopy_mesh_step10_link4_num4.obj.urdf (robot description, URDF)
Before this commit: robot zonopy_mesh_step10_link4_num4.obj, 1 links, 0 joints
Links:
- removed link 
- added link link0, mass 0; collision mesh filename=zonopy_mesh_step10_link4_num4.obj; visual mesh filename=zonopy_mesh_step10_link4_num4.obj scale=1.0 1.0 1.0

File: zonotope/meshes/zonopy_mesh_step10_link5_num1.obj.urdf (robot description, URDF)
Before this commit: robot zonopy_mesh_step10_link5_num1.obj, 1 links, 0 joints
Links:
- removed link 
- added link link0, mass 0; collision mesh filename=zonopy_mesh_step10_link5_num1.obj; visual mesh filename=zonopy_mesh_step10_link5_num1.obj scale=1.0 1.0 1.0

File: zonotope/meshes/zonopy_mesh_step10_link5_num2.obj.urdf (robot description, URDF)
Before this commit: robot zonopy_mesh_step10_link5_num2.obj, 1 links, 0 joints
Links:
- removed link 
- added link link0, mass 0; collision mesh filename=zonopy_mesh_step10_link5_num2.obj; visual mesh filename=zonopy_mesh_step10_link5_num2.obj scale=1.0 1.0 1.0

File: zonotope/meshes/zonopy_mesh_step10_link5_num3.obj.urdf (robot description, URDF)
Before this commit: robot zonopy_mesh_step10_link5_num3.obj, 1 links, 0 joints
Links:
- removed link 
- added link link0, mass 0; collision mesh filename=zonopy_mesh_step10_link5_num3.obj; visual mesh filename=zonopy_mesh_step10_link5_num3.obj scale=1.0 1.0 1.0
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