Commit message: format directories

File: assets/kinova_gen3_7dof/kinova_with_robotiq_85.urdf (robot description, URDF)
Before this commit: robot GEN3_URDF_V12, 10 links, 9 joints
Links:
- link Base_Link: geometry collision mesh filename=meshes/base_link.stl; visual mesh filename=meshes/base_link.obj
- link Bracelet_Link: geometry collision mesh filename=meshes/bracelet_no_vision_link.stl; visual mesh filename=meshes/bracelet_no_vision_link.obj
- link ForeArm_Link: geometry collision mesh filename=meshes/forearm_link.stl; visual mesh filename=meshes/forearm_link.obj
- link HalfArm1_Link: geometry collision mesh filename=meshes/half_arm_1_link.stl; visual mesh filename=meshes/half_arm_1_link.obj
- link HalfArm2_Link: geometry collision mesh filename=meshes/half_arm_2_link.stl; visual mesh filename=meshes/half_arm_2_link.obj
- link Shoulder_Link: geometry collision mesh filename=meshes/shoulder_link.stl; visual mesh filename=meshes/shoulder_link.obj
- link SphericalWrist1_Link: geometry collision mesh filename=meshes/spherical_wrist_1_link.stl; visual mesh filename=meshes/spherical_wrist_1_link.obj
- link SphericalWrist2_Link: geometry collision mesh filename=meshes/spherical_wrist_2_link.stl; visual mesh filename=meshes/spherical_wrist_2_link.obj
