Commit message: modify kinova_with_gripper_dumbbell.urdf

File: assets/kinova_gen3_7dof/kinova_with_gripper_dumbbell.urdf (robot description, URDF)
Before this commit: robot GEN3_URDF_V12, 22 links, 21 joints
Joints:
- joint gripper_left_coupler_joint: origin xyz=0.031486 -0.0040855 0 rpy=3.1416 0 1.5707 -> xyz=0.031486 -0.0040855 0 rpy=3.1416 0 1.56
- joint gripper_left_driver_joint: origin xyz=-0.030601 -0.054792 0 rpy=0 0 -1.5707 -> xyz=-0.030601 -0.054792 0 rpy=0 0 -1.5
- joint gripper_right_coupler_joint: origin xyz=0.031486 -0.0040855 0 rpy=0 0 -1.5707 -> xyz=0.031486 -0.0040855 0 rpy=0 0 -1.53
- joint gripper_right_driver_joint: origin xyz=0.030601 -0.054792 0 rpy=3.1416 0 -1.5707 -> xyz=0.030601 -0.054792 0 rpy=3.1416 0 -1.5

Commit message: modify urdf; add test scripts

File: assets/kinova_gen3_7dof/kinova_with_gripper_dumbbell.urdf (robot description, URDF)
Before this commit: robot GEN3_URDF_V12, 22 links, 21 joints
Joints:
- joint dumbbell_joint: origin xyz=0 0 0.170 rpy=0 0 0 -> xyz=0 0 0.150 rpy=0 0 0

Commit message: update urdf; update test script

File: assets/kinova_gen3_7dof/kinova_with_gripper_dumbbell.urdf (robot description, URDF)
Before this commit: robot GEN3_URDF_V12, 22 links, 21 joints
Joints:
- joint dumbbell_joint: origin xyz=0 0 0.150 rpy=0 0 0 -> xyz=0 0 0.150 rpy=1.571 0 0

File: assets/kinova_gen3_7dof/kinova_with_gripper_dumbbell_approx.urdf (robot description, URDF)
Before this commit: robot GEN3_URDF_V12, 11 links, 10 joints
Links:
- removed link Tool_Frame
- removed link gripper_base_approx
- added link gripper_base
- added link gripper_dumbbell_approx, mass 1.7215; collision mesh filename=../objects/cube.obj; visual mesh filename=../objects/cube.obj
Joints:
- removed joint Tool
- added joint gripper_dumbbell_joint: type fixed, parent gripper_base, child gripper_dumbbell_approx, origin xyz=0.0 -0.10155 0 rpy=0.0 0.0 0.0
- joint gripper_base_joint: child gripper_base_approx -> gripper_base
