Commit message: modify base link mesh name; improve debug_script.m

File: assets/kinova_gen3_7dof/kinova_with_dumbbell.urdf (robot description, URDF)
Before this commit: robot GEN3_URDF_V12, 10 links, 9 joints
Links:
- link Base_Link: geometry collision mesh filename=meshes/base_link_kinova.stl; visual mesh filename=meshes/base_link_kinova.obj

File: assets/kinova_gen3_7dof/kinova_with_gripper_dumbbell.urdf (robot description, URDF)
Before this commit: robot GEN3_URDF_V12, 22 links, 21 joints
Links:
- link Base_Link: geometry collision mesh filename=meshes/base_link_kinova.stl; visual mesh filename=meshes/base_link_kinova.obj

File: assets/kinova_gen3_7dof/kinova_with_gripper_dumbbell_approx.urdf (robot description, URDF)
Before this commit: robot GEN3_URDF_V12, 11 links, 10 joints
Links:
- link Base_Link: geometry collision mesh filename=meshes/base_link_kinova.stl; visual mesh filename=meshes/base_link_kinova.obj
