Commit message: new demo complete: kinova with table

File: assets/kinova_w_tray/CC_Kinova_combined_wo_cube.urdf (robot description, URDF)
Before this commit: robot gen3_robotiq_2f_85, 10 links, 9 joints
Links:
- link base: geometry collision mesh filename=.\meshes\base_link.STL; visual mesh filename=.\meshes\base_link.obj
- link bracelet_link: geometry collision mesh filename=.\meshes\bracelet_with_vision_link.STL; visual mesh filename=.\meshes\bracelet_with_vision_link.obj
- link forearm_link: geometry collision mesh filename=.\meshes\forearm_link.STL; visual mesh filename=.\meshes\forearm_link.obj
- link gripper_base: geometry collision mesh filename=.\meshes\base_of_gripper.STL; visual mesh filename=.\meshes\base_of_gripper.obj
- link half_arm_1_link: geometry collision mesh filename=.\meshes\half_arm_1_link.STL; visual mesh filename=.\meshes\half_arm_1_link.obj
- link half_arm_2_link: geometry collision mesh filename=.\meshes\half_arm_2_link.STL; visual mesh filename=.\meshes\half_arm_2_link.obj
- link shoulder_link: geometry collision mesh filename=.\meshes\shoulder_link.STL; visual mesh filename=.\meshes\shoulder_link.obj
- link spherical_wrist_1_link: geometry collision mesh filename=.\meshes\spherical_wrist_1_link.STL; visual mesh filename=.\meshes\spherical_wrist_1_link.obj
- link spherical_wrist_2_link: geometry collision mesh filename=.\meshes\spherical_wrist_2_link.STL; visual mesh filename=.\meshes\spherical_wrist_2_link.obj
- link waiter_tray_link: geometry collision mesh filename=.\meshes\plate_shifted_scaled_origin_v3.STL; visual mesh filename=.\meshes\plate_shifted_scaled_origin_v3.obj
