Commit message: generate new figures

File: assets/kinova_w_tray/CC_Kinova_combined.urdf (robot description, URDF)
Before this commit: robot gen3_robotiq_2f_85, 11 links, 10 joints
Links:
- added link gripper_left_coupler, mass 0.0273093985570947; collision mesh filename=meshes/left_coupler.STL; visual mesh filename=meshes/left_coupler.STL
- added link gripper_left_driver, mass 0.0184906489414316; collision mesh filename=meshes/left_driver.STL; visual mesh filename=meshes/left_driver.STL
- added link gripper_left_follower, mass 0.0195548943464751; collision mesh filename=meshes/left_follower.STL; visual mesh filename=meshes/left_follower.STL
- added link gripper_left_pad, mass 0.0112846745192961; collision mesh filename=meshes/left_pad.STL; visual mesh filename=meshes/left_pad.STL
- added link gripper_left_spring_link, mass 0.0299513316731757; collision mesh filename=meshes/left_spring_link.STL; visual mesh filename=meshes/left_spring_link.STL
- added link gripper_right_coupler, mass 0.0273093985570947; collision mesh filename=meshes/right_coupler.STL; visual mesh filename=meshes/right_coupler.STL
- added link gripper_right_driver, mass 0.0184906489409923; collision mesh filename=meshes/right_driver.STL; visual mesh filename=meshes/right_driver.STL
- added link gripper_right_follower, mass 0.0195548943464751; collision mesh filename=meshes/right_follower.STL; visual mesh filename=meshes/right_follower.STL
- added link gripper_right_pad, mass 0.0112846745192962; collision mesh filename=meshes/right_pad.STL; visual mesh filename=meshes/right_pad.STL
- added link gripper_right_spring_link, mass 0.029951; collision mesh filename=meshes/right_spring_link.STL; visual mesh filename=meshes/right_spring_link.STL
Joints:
- added joint gripper_left_coupler_joint: type fixed, parent gripper_left_driver, child gripper_left_coupler, origin xyz=0.031486 -0.0040855 0 rpy=3.1416 0 1.5707, axis 0 0 1, limit lower=0.13 upper=0.79 effort=0 velocity=0
- added joint gripper_left_driver_joint: type fixed, parent gripper_base, child gripper_left_driver, origin xyz=-0.030601 -0.054792 0 rpy=0 0 -1.5707, axis 0 0 1, limit lower=-3.1416 upper=3.1416 effort=150 velocity=0
- added joint gripper_left_follower_joint: type fixed, parent gripper_left_coupler, child gripper_left_follower, origin xyz=-0.0061148 0.047125 0 rpy=0 0 0, axis 0 0 1, limit lower=-3.1416 upper=3.1416 effort=0 velocity=0
- added joint gripper_left_pad_joint: type fixed, parent gripper_left_follower, child gripper_left_pad, origin xyz=0.018903 0.032265 0 rpy=0 0 -1.5708, axis 0 0 0
- added joint gripper_left_spring_link_joint: type fixed, parent gripper_base, child gripper_left_spring_link, origin xyz=-0.0127 -0.061307 0 rpy=3.1416 0 -0.392699, axis 0 0 1, limit lower=-0.7854 upper=0 effort=0 velocity=0
- added joint gripper_right_coupler_joint: type fixed, parent gripper_right_driver, child gripper_right_coupler, origin xyz=0.031486 -0.0040855 0 rpy=0 0 -1.5707, axis 0 0 -1, limit lower=0.13 upper=0.79 effort=0 velocity=0
- added joint gripper_right_driver_joint: type fixed, parent gripper_base, child gripper_right_driver, origin xyz=0.030601 -0.054792 0 rpy=3.1416 0 -1.5707, axis 0 0 1, limit lower=-3.1416 upper=3.1416 effort=150 velocity=0
- added joint gripper_right_follower_joint: type fixed, parent gripper_right_coupler, child gripper_right_follower, origin xyz=-0.0061148 0.047125 0 rpy=3.1416 0 3.1416, axis 0 0 1, limit lower=-3.1416 upper=3.1416 effort=0 velocity=0
- added joint gripper_right_pad_joint: type fixed, parent gripper_right_follower, child gripper_right_pad, origin xyz=0.024903 0.032264 0 rpy=3.1416 0 -1.5708, axis 0 0 0
- added joint gripper_right_spring_link_joint: type fixed, parent gripper_base, child gripper_right_spring_link, origin xyz=0.0127 -0.061307 0 rpy=3.1416 0 0.392699, axis 0 0 1, limit lower=0 upper=0.7854 effort=0 velocity=0
