Commit message: found a way to modify obstacle scale in pybullet: parse and edit directly

File: assets/objects/cube_small_zero.urdf (robot description, URDF)
Before this commit: robot cube.urdf, 1 links, 0 joints
Links:
- link baseLink: geometry collision box size=0.2 0.2 0.2; visual mesh filename=cube.obj scale=0.2 0.2 0.2
